File: modules/output-register/m1-output-reg.sch (EAGLE design)
At the start: 40 parts, among them U1 555, U2 74HCT109D, U3 74LS139AD, U4 74LS273NS, U5 74LS08, U6 28C64

Commit message: Various updates
Other:
- note added: "Add mode switch"
Changed lines of the file:
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@@
 <wire x1="94.996" y1="53.848" x2="93.98" y2="52.578" width="0.1524" layer="150"/>
 <wire x1="93.98" y1="52.578" x2="92.964" y2="53.848" width="0.1524" layer="150"/>
+<text x="30.48" y="106.68" size="3.81" layer="150">Add mode switch</text>
 </plain>
 <instances>
