File: modules/registers/m1-data-register-a.brd (EAGLE design)
At the start: 42 x 30 mm, 44 parts, among them U1 74LS245NS, U2 74LS173AD, U3 74LS173AD

Commit message: Various updates
Parts:
- C1, C2, C3: value (none) -> 0.1uF
Changed lines of the file:
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@@
 <?xml version="1.0" encoding="utf-8"?>
 <!DOCTYPE eagle SYSTEM "eagle.dtd">
-<eagle version="9.5.2">
+<eagle version="9.6.1">
 <drawing>
 <settings>
@@
 </layers>
 <board>
-<fusionsync huburn="a.cGVyc29uYWw6dWUyYmRlZGJl" projecturn="a.cGVyc29uYWw6dWUyYmRlZGJlIzIwMTgwNTA0MTMwNTkwMzU2" f3durn="urn:adsk.wipprod:dm.lineage:t5Up-ix5QhOrgsyVkisISg" pcbguid="899eb2d3-baae-49c1-a65f-7f97990e736e" lastpulledtime="" lastsyncedchangeguid="0a45ebb6-d4d9-1a97-533b-fb940c91d080"/>
+<fusionsync huburn="a.cGVyc29uYWw6dWUyYmRlZGJl" projecturn="a.cGVyc29uYWw6dWUyYmRlZGJlIzIwMTgwNTA0MTMwNTkwMzU2" f3durn="urn:adsk.wipprod:dm.lineage:t5Up-ix5QhOrgsyVkisISg" pcbguid="899eb2d3-baae-49c1-a65f-7f97990e736e" lastpulledtime="" lastsyncedchangeguid="0a45ebb6-d4d9-1a97-533b-fb940c91d080" latestrevisionid="" lastsyncedrevisionid="" lastboardhashguid="" lastpushedtime="" linktopcb3d="%12"/>
 <plain>
 <wire x1="0" y1="1.5" x2="1.5" y2="0" width="0.01" layer="20"/>
@@
 <attribute name="VALUE" x="29" y="8.762" size="0.762" layer="21" align="center"/>
 </element>
-<element name="C1" library="rlc" library_urn="urn:adsk.eagle:library:4192893" package="0603-CAP" package3d_urn="urn:adsk.eagle:package:4193021/2" value="" x="10.538" y="28.079" smashed="yes" rot="R270">
+<element name="C1" library="rlc" library_urn="urn:adsk.eagle:library:4192893" package="0603-CAP" package3d_urn="urn:adsk.eagle:package:4193021/2" value="0.1uF" x="10.538" y="28.079" smashed="yes" rot="R270">
 <attribute name="NAME" x="10.481" y="26.401" size="0.8128" layer="125" font="vector" ratio="15" rot="R270" align="center-left"/>
 <attribute name="VALUE" x="10.538" y="28.079" size="0.2" layer="27" rot="R270" align="center"/>
 </element>
-<element name="C2" library="rlc" library_urn="urn:adsk.eagle:library:4192893" package="0603-CAP" package3d_urn="urn:adsk.eagle:package:4193021/2" value="" x="10.94" y="8.7" smashed="yes" rot="R270">
+<element name="C2" library="rlc" library_urn="urn:adsk.eagle:library:4192893" package="0603-CAP" package3d_urn="urn:adsk.eagle:package:4193021/2" value="0.1uF" x="10.94" y="8.7" smashed="yes" rot="R270">
 <attribute name="NAME" x="10.86" y="10.4" size="0.8128" layer="125" font="vector" ratio="15" rot="R90" align="center-left"/>
 <attribute name="VALUE" x="10.94" y="8.7" size="0.2" layer="27" rot="R270" align="center"/>
 </element>
-<element name="C3" library="rlc" library_urn="urn:adsk.eagle:library:4192893" package="0603-CAP" package3d_urn="urn:adsk.eagle:package:4193021/2" value="" x="22.96" y="8.7" smashed="yes" rot="R270">
+<element name="C3" library="rlc" library_urn="urn:adsk.eagle:library:4192893" package="0603-CAP" package3d_urn="urn:adsk.eagle:package:4193021/2" value="0.1uF" x="22.96" y="8.7" smashed="yes" rot="R270">
 <attribute name="NAME" x="23" y="10.36" size="0.8128" layer="125" font="vector" ratio="15" rot="R90" align="center-left"/>
 <attribute name="VALUE" x="22.96" y="8.7" size="0.2" layer="27" rot="R270" align="center"/>
